File: PCB/AstroPix5/astropix_v5.kicad_sch (KiCad schematic)
At the start: 37 parts, among them J1 pcie_GECCO, J10 SPI_right, J11 HV, J2 Conn_02x04_Odd_Even, J4 SFOut, J6 HV_in_external, J8 HBOut, J9 SPI_left, U1 AstroPix4_split_powerring

Commit message: modif v5
Parts:
- removed C1, C11, C8: 1nF, Capacitor_SMD:C_0603_1608Metric, symbol Device:C
- removed C10, C14, C15: 10uF, Capacitor_SMD:C_0603_1608Metric, symbol Device:C
- removed C13, C2, C9: .1uF, Capacitor_SMD:C_0603_1608Metric, symbol Device:C
- removed C4: 1nF, Capacitor_SMD:C_1210_3225Metric, symbol Device:C
- removed C6: .1uF, Capacitor_SMD:C_1210_3225Metric, symbol Device:C
- removed FID1, FID2: Fiducial, Fiducial:Fiducial_1mm_Mask2mm, symbol Mechanical:Fiducial
- removed H1, H2: MountingHole, MountingHole:MountingHole_3.2mm_M3, symbol Mechanical:MountingHole
- removed H3: bonder, astropix:bonder, symbol astropix:bonder
- removed J1: pcie_GECCO, astropix:pcie_astropix, symbol astropix:pcie_GECCO
- removed J10: SPI_right, Connector_PinHeader_2.54mm:PinHeader_1x06_P2.54mm_Vertical, symbol Connector_Generic:Conn_01x06
- removed J11: HV, Connector_PinHeader_2.54mm:PinHeader_1x05_P2.54mm_Vertical, symbol Connector_Generic:Conn_01x05
- removed J2: Conn_02x04_Odd_Even, Connector_PinHeader_2.54mm:PinHeader_2x04_P2.54mm_Vertical, symbol Connector_Generic:Conn_02x04_Odd_Even
- removed J4: SFOut, Connector_Coaxial:SMA_Molex_73251-2200_Horizontal, symbol Connector:Conn_Coaxial
- removed J6: HV_in_external, Connector_Coaxial:SMA_Molex_73251-2200_Horizontal, symbol Connector:Conn_Coaxial
- removed J8: HBOut, Connector_Coaxial:SMA_Molex_73251-2200_Horizontal, symbol Connector:Conn_Coaxial
- removed J9: SPI_left, Connector_PinHeader_2.54mm:PinHeader_1x06_P2.54mm_Vertical, symbol Connector_Generic:Conn_01x06
- removed JP1: VDD_JP, Connector_PinHeader_2.54mm:PinHeader_1x03_P2.54mm_Vertical, symbol Jumper:Jumper_3_Bridged12
- removed Logo1: KIT_logo, astropix:logo, symbol astropix:KIT_logo
- removed Logo2, Logo3: HV_logo, astropix:hv, symbol astropix:HV_logo
- removed R1, R2: 2.2k, Resistor_SMD:R_0603_1608Metric, symbol Device:R
- removed R10, R13, R14, R17, R18: 22, Resistor_SMD:R_0402_1005Metric, symbol Device:R
- removed R12: 1k, Resistor_SMD:R_0603_1608Metric, symbol Device:R
- removed U1: AstroPix4_split_powerring, astropix:AstroPix4, symbol astropix:AstroPix4_split_powerring
- added C12, C20, C21: 10uF, Capacitor_SMD:C_0603_1608Metric, symbol Device:C
- added C16, C17, C5: 1nF, Capacitor_SMD:C_0603_1608Metric, symbol Device:C
- added C18, C19, C7: .1uF, Capacitor_SMD:C_0603_1608Metric, symbol Device:C
- added C22: 1nF, Capacitor_SMD:C_1210_3225Metric, symbol Device:C
- added C23: .1uF, Capacitor_SMD:C_1210_3225Metric, symbol Device:C
- added C3: 100 nF, Capacitor_SMD:C_0603_1608Metric, symbol Device:C
- added FID3, FID4: Fiducial, Fiducial:Fiducial_1mm_Mask2mm, symbol Mechanical:Fiducial
- added H4, H5: MountingHole, MountingHole:MountingHole_3.2mm_M3, symbol Mechanical:MountingHole
- added H6: bonder, astropix:bonder, symbol astropix:bonder
- added J12: Measures_Analog, symbol Connector_Generic:Conn_01x04
- added J13: pcie_GECCO, astropix:pcie_astropix, symbol astropix:pcie_GECCO_v2
- added J14: Bias, symbol Connector_Generic:Conn_02x06_Odd_Even
- added J15: HV_in_external, Connector_Coaxial:SMA_Molex_73251-2200_Horizontal, symbol Connector:Conn_Coaxial
- added J17: SPI_right, Connector_PinHeader_2.54mm:PinHeader_1x06_P2.54mm_Vertical, symbol Connector_Generic:Conn_01x06
- added J18: Measures_Digital, symbol Connector_Generic:Conn_01x04
- added J3: SPI_left, Connector_PinHeader_2.54mm:PinHeader_1x06_P2.54mm_Vertical, symbol Connector_Generic:Conn_01x06
- added J5: HBOut, Connector_Coaxial:SMA_Molex_73251-2200_Horizontal, symbol Connector:Conn_Coaxial
- added J7: SFOut, Connector_Coaxial:SMA_Molex_73251-2200_Horizontal, symbol Connector:Conn_Coaxial
- added JP2: VDD_JP, Connector_PinHeader_2.54mm:PinHeader_1x03_P2.54mm_Vertical, symbol Jumper:Jumper_3_Bridged12
- added Logo4: KIT_logo, astropix:logo, symbol astropix:KIT_logo
- added Logo5, Logo6: HV_logo, astropix:hv, symbol astropix:HV_logo
- added R11, R15, R7, R8: 10k, Resistor_SMD:R_0603_1608Metric, symbol Device:R
- added R3, R6: 0, Resistor_SMD:R_0603_1608Metric, symbol Device:R
- added R4, R5: 2.2k, Resistor_SMD:R_0603_1608Metric, symbol Device:R
- added R9: 1k, Resistor_SMD:R_0603_1608Metric, symbol Device:R
- added U2: AstroPix5_split_powerring, astropix:AstroPix5, symbol astropix:AstroPix5_split_powerring_1
Connections:
- net DigInj: now also J13.B40 (FMC_LA16_P), R8.2, U2.B93 (DigInj)
- net GND: now also C12.2, C16.2, C17.2, C18.2, C19.2, C20.2, C21.2, C22.1, C23.1, C3.1, C5.2, C7.2, J12.4 (Pin_4), J13.A11 (GND), J13.B11 (GND), J14.11 (Pin_11), J15.2 (Ext), J17.6 (Pin_6), J18.4 (Pin_4), J3.6 (Pin_6), J5.2 (Ext), J7.2 (Ext), R11.1, R15.1, R4.2, R5.2, R7.1, R8.1, U2.B100 (gnda!), U2.B101 (gnda!), U2.B103 (gnda!), U2.B105 (gnda!), U2.B110 (gnd!), U2.B12 (gnda!), U2.B14 (gnda!), U2.B16 (gnda!), U2.B2 (gnd!), U2.B27 (gnd!), U2.B32 (gnd!), U2.B39 (gnd!), U2.B45 (gnd!), U2.B59 (gnd!), U2.B61 (gnda!), U2.B65 (gnda!), U2.B70 (gnda!), U2.B73 (gnda!), U2.B75 (gnda!), U2.B8 (gnd!), U2.B83 (gnda!), U2.B89 (gnda!), U2.B9 (gnd!), U2.B92 (gnda!), U2.B95 (gnd!)
- net HV_in_ext: now also J15.1 (In), R9.1
- net Inj: now also J13.A28 (C3_1), R7.2, U2.B72 (Inj)
- net POW4_in: now also J13.B5 (POW4), J13.B6 (POW4), JP2.3 (B)
- net VDD: now also C12.1, C5.1, C7.1, J18.1 (Pin_1), JP2.2 (C), U2.B1 (vdd!), U2.B10 (vdd!), U2.B109 (vdd!), U2.B11 (vdd!), U2.B26 (vdd!), U2.B44 (vdd!), U2.B58 (vdd!), U2.B94 (vdd!)
- net VDD18_in: now also J13.B3 (VDD18), J13.B4 (VDD18), JP2.1 (A)
- net VDDA: now also C17.1, C19.1, C21.1, J13.B7 (POW6), J13.B8 (POW6), R3.1, U2.B102 (vdda!), U2.B104 (vdda!), U2.B106 (vdda!), U2.B13 (vdda!), U2.B15 (vdda!), U2.B17 (vdda!), U2.B60 (vdda!), U2.B64 (vdda!), U2.B71 (vdda!), U2.B76 (vdda!), U2.B82 (vdda!), U2.B88 (vdda!), U2.B91 (vdda!), U2.B99 (vdda!)
- net VSSA: now also C16.1, C18.1, C20.1, J13.A5 (VSSA), J13.A6 (VSSA), U2.B107 (vssa!), U2.B108 (vssa!), U2.B18 (vssa!), U2.B19 (vssa!), U2.B62 (vssa!), U2.B63 (vssa!), U2.B80 (vssa!), U2.B87 (vssa!), U2.B90 (vssa!)
- net Vtemp1: now also J12.1 (Pin_1), U2.B84 (Vtemp1)
- net Vtemp2: now also J12.2 (Pin_2), U2.B85 (Vtemp2)
- net cascpix: now also J14.6 (Pin_6), U2.B86 (cascpix)
- net hold: now also J13.B18 (FMC_LA22_P), U2.B49 (hold)
- net interrupt: now also J13.B20 (FMC_LA20_P), U2.B46 (interrupt)
- net pamp: now also J14.3 (Pin_3), U2.B67 (pamp)
- net pload: now also J14.7 (Pin_7), U2.B69 (pload)
- net res_n: now also J13.B21 (FMC_LA20_N), U2.B47 (res_n)
- net suba: now also C22.2, C23.2, R9.2, U2.B4 (sub!), U2.B5 (sub!)
- net timestamp_clk: now also J13.B19 (FMC_LA22_N), U2.B41 (timestamp_clk)
- new net: R3.2, U2.B6 (dnring)
- new net: C3.2, U2.B20 (VGateComp!)
- new net: R6.1, U2.B97 (vminusout)
- new net Clk20_Ext_N: U2.B43 (Clk20_Ext_N)
- new net Clk20_Ext_P: U2.B42 (Clk20_Ext_P)
- new net Enable_SPI_diff: J13.A45 (FMC_LA11_N), R15.2, U2.B25 (Enable_SPI_diff)
- new net HBOut: J5.1 (In), R4.1, U2.B40 (HBOut)
- new net SPI_CLK_N: J13.A51 (FMC_LA06_N), U2.B36 (SPI_CLK_N)
- new net SPI_CLK_P: J13.A50 (FMC_LA06_P), U2.B35 (SPI_CLK_P)
- new net SPI_CSN_N: J13.A53 (FMC_LA04_N), U2.B38 (SPI_CSN_N)
- new net SPI_CSN_P: J13.A52 (FMC_LA04_P), U2.B37 (SPI_CSN_P)
- new net SPI_MISO0_N: J13.B51 (FMC_LA05_N), U2.B31 (SPI_MISO0_N)
- new net SPI_MISO0_P: J13.B50 (FMC_LA05_P), U2.B30 (SPI_MISO0_P)
- new net SPI_MISO1_N: J13.B49 (FMC_LA08_N), U2.B29 (SPI_MISO1_N)
- new net SPI_MISO1_P: J13.B48 (FMC_LA08_P), U2.B28 (SPI_MISO1_P)
- new net SPI_MOSI_N: J13.A49 (FMC_LA07_N), U2.B34 (SPI_MOSI_N)
- new net SPI_MOSI_P: J13.A48 (FMC_LA07_P), U2.B33 (SPI_MOSI_P)
- new net SPI_left_CLK: J13.A17 (FMC_LA23_N), J3.4 (Pin_4), U2.L4 (SPI_left_CLK)
- new net SPI_left_CSN: J13.A16 (FMC_LA23_P), J3.5 (Pin_5), U2.L5 (SPI_left_CSN)
- new net SPI_left_MISO0: J13.A19 (FMC_LA21_N), J3.2 (Pin_2), U2.L2 (SPI_left_MISO0)
- new net SPI_left_MISO1: J13.A18 (FMC_LA21_P), J3.3 (Pin_3), U2.L1 (SPI_left_MISO1)
- new net SPI_left_MOSI: J13.A20 (FMC_LA19_P), J3.1 (Pin_1), U2.L3 (SPI_left_MOSI)
- new net SPI_right_CLK: J13.A40 (FMC_LA15_P), J17.1 (Pin_1), U2.R2 (SPI_right_CLK)
- new net SPI_right_CSN: J13.A43 (FMC_LA13_N), J17.4 (Pin_4), U2.R1 (SPI_right_CSN)
- new net SPI_right_MISO0: J13.A42 (FMC_LA13_P), J17.3 (Pin_3), U2.R4 (SPI_right_MISO<0>)
- new net SPI_right_MISO1: J13.A41 (FMC_LA15_N), J17.2 (Pin_2), U2.R5 (SPI_right_MISO<1>)
- new net SPI_right_MOSI: J13.A44 (FMC_LA11_P), J17.5 (Pin_5), U2.R3 (SPI_right_MOSI)
- new net SR_ck1: J13.A24 (C2_1), J13.B42 (FMC_LA14_P), U2.B50 (SR_ck1)
- new net SR_ck2: J13.A25 (C2_2), J13.B43 (FMC_LA14_N), U2.B51 (SR_ck2)
- new net SR_ldpatgen: J13.A26 (C2_5), U2.B56 (SR_ldpatgen)
- new net SR_ldtdac: J13.A21 (FMC_LA19_N), U2.B55 (SR_ldtdac)
- new net SR_load: J13.B24 (C2_4), J13.B44 (FMC_LA12_P), U2.B52 (SR_load)
- new net SR_out_0D: J13.B26 (C2_8), U2.B21 (SR_out_OD)
- new net SR_out_CK1: J13.B27 (C2_7), U2.B22 (SR_out_CK1)
- new net SR_rb: J13.A23 (FMC_LA17_CC_N), U2.B54 (SR_rb)
- new net SR_sin: J13.B25 (C2_3), J13.B45 (FMC_LA12_N), U2.B53 (SR_sin)
- new net SR_sout: J13.A22 (FMC_LA17_CC_P), U2.B57 (SR_sout)
- new net ThPix: J13.B34 (C4_8), J14.2 (Pin_2), U2.B74 (ThPix)
- new net VCasc2!: J13.B33 (C4_3), J14.4 (Pin_4), U2.B81 (VCasc2!)
- new net VPBias!: J14.1 (Pin_1), U2.B66 (VPBias!)
- new net ampout: J7.1 (In), R5.1, U2.B77 (ampout)
- new net blpix: J13.B32 (C4_4), J14.5 (Pin_5), U2.B68 (blpix)
- new net clk20_Ext_N: J13.B17 (FMC_LA24_N)
- new net clk20_Ext_P: J13.B16 (FMC_LA24_P)
- new net pll_clk: J18.2 (Pin_2), U2.B24 (pll_clk)
- new net syncres: J13.B22 (FMC_LA18_CC_P), R11.2, U2.B48 (syncres)
- new net vminuspix: J13.B35 (C4_7), J13.B39 (C5_7), R6.2, U2.B98 (vminuspix)
- new net vminusref: J14.8 (Pin_8), U2.B96 (vminusref)
- new net vpDel: J14.9 (Pin_9), U2.B23 (vpDel)
- no-connect marks 55 -> 51
Other:
- note removed: "Connect dnring to 1.8V to collect leakage current"
- note removed: "Pullup in fpga"
- note removed: "internal switchable 100Ohm diff termination"

Commit message: Schematic draft 2
Parts:
- removed J7: SFOut, Connector_Coaxial:SMA_Molex_73251-2200_Horizontal, symbol Connector:Conn_Coaxial
- removed R11, R15, R7, R8: 10k, Resistor_SMD:R_0603_1608Metric, symbol Device:R
- removed R3: 0, Resistor_SMD:R_0603_1608Metric, symbol Device:R
- removed R4, R5: 2.2k, Resistor_SMD:R_0603_1608Metric, symbol Device:R
- added J2: Conn_01x05, symbol Connector_Generic:Conn_01x05
- added JP1, JP3: Jumper_3_Bridged12, symbol Jumper:Jumper_3_Bridged12
- added JP4, JP5: Jumper_2_Bridged, symbol Jumper:Jumper_2_Bridged
- added R1: 10k, Resistor_SMD:R_0603_1608Metric, symbol Device:R
- added TP1, TP2: TestPoint, symbol Connector:TestPoint
Connections:
- net GND: now also J3.1 (Pin_1), JP3.1 (A); no longer J3.6 (Pin_6)
- net SPI_left_CLK: now also J3.5 (Pin_5); no longer J3.4 (Pin_4)
- net SPI_left_CSN: now also J3.4 (Pin_4); no longer J3.5 (Pin_5)
- net SPI_left_MOSI: now also J3.6 (Pin_6); no longer J3.1 (Pin_1)
- net SPI_right_CLK: now also J17.2 (Pin_2); no longer J17.1 (Pin_1)
- net SPI_right_CSN: now also J17.3 (Pin_3); no longer J17.4 (Pin_4)
- net SPI_right_MISO0: now also J17.4 (Pin_4); no longer J17.3 (Pin_3)
- net SPI_right_MISO1: now also J17.5 (Pin_5); no longer J17.2 (Pin_2)
- net SPI_right_MOSI: now also J17.1 (Pin_1); no longer J17.5 (Pin_5)
- net ThPix: no longer J14.2 (Pin_2), U2.B74 (ThPix)
- net VCasc2!: no longer J14.4 (Pin_4), U2.B81 (VCasc2!)
- net VDD: now also R1.1
- net VDDA: now also JP3.3 (B)
- net blpix: no longer J14.5 (Pin_5), U2.B68 (blpix)
- net interrupt: now also R1.2
- net at U2.B6 (dnring): now also JP3.2 (C)
- net at J14.10 (Pin_10): now also U2.B86 (cascpix)
- net at J14.12 (Pin_12): now also U2.B96 (vminusref)
- net at U2.B3 (chipring): now also JP5.2 (B)
- net at U2.B7 (pring_pixel): now also JP4.2 (B)
- net at U2.B78 (Qdac<0>): now also TP1.1
- net at U2.B79 (Qdac<1>): now also TP2.1
- net at U2.L10 (pring0): now also J2.1 (Pin_1)
- net at U2.L6 (pring4): now also J2.5 (Pin_5)
- net at U2.L7 (pring3): now also J2.4 (Pin_4)
- net at U2.L8 (pring2): now also J2.3 (Pin_3)
- net at U2.L9 (pring1): now also J2.2 (Pin_2)
- net HBOut: no longer names the net of U2.B40 (HBOut)
- net HBOut: now also JP1.3 (B); no longer J5.1 (In)
- net VPBias!: no longer names the net of J14.1 (Pin_1)
- net VPBias!: now also U2.B67 (pamp); no longer U2.B66 (VPBias!)
- net Vtemp1: no longer names the net of J12.1 (Pin_1), U2.B84 (Vtemp1)
- net Vtemp2: no longer names the net of J12.2 (Pin_2), U2.B85 (Vtemp2)
- net ampout: no longer names the net of U2.B77 (ampout)
- net ampout: now also JP1.1 (A)
- net cascpix: no longer names the net of J14.6 (Pin_6)
- net cascpix: now also U2.B74 (ThPix); no longer U2.B86 (cascpix)
- net pamp: no longer names the net of J14.3 (Pin_3)
- net pamp: now also U2.B66 (VPBias!); no longer U2.B67 (pamp)
- net pll_clk: no longer names the net of J18.2 (Pin_2), U2.B24 (pll_clk)
- net pload: no longer names the net of U2.B69 (pload)
- net pload: now also J14.4 (Pin_4); no longer J14.7 (Pin_7)
- net suba: no longer names the net of C22.2, C23.2, R9.2, U2.B4 (sub!), U2.B5 (sub!)
- net suba: now also JP4.1 (A), JP5.1 (A)
- net vminusref: no longer names the net of J14.8 (Pin_8)
- net vminusref: now also U2.B81 (VCasc2!); no longer U2.B96 (vminusref)
- net vpDel: no longer names the net of U2.B23 (vpDel)
- net vpDel: now also J14.5 (Pin_5); no longer J14.9 (Pin_9)
- new net: J14.2 (Pin_2), U2.B68 (blpix)
- new net: J5.1 (In), JP1.2 (C)
- no-connect marks 51 -> 46
Other:
- company: Nicolas Striebig, KIT IPE -> Ilona Munnich, KIT IPE
- title: AstroPix4 Carrier -> AstroPix5 Carrier
- moved on the sheet: C12, C16, C17, C18, C19, C20, C21, C22, C23, C3, C5, C7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

Commit message: Small modifications in schematic and layout finished
Parts:
- removed C12, C20, C21: 10uF, Capacitor_SMD:C_0603_1608Metric, symbol Device:C
- removed C16, C17, C5: 1nF, Capacitor_SMD:C_0603_1608Metric, symbol Device:C
- removed C18, C19, C7: .1uF, Capacitor_SMD:C_0603_1608Metric, symbol Device:C
- removed C22: 1nF, Capacitor_SMD:C_1210_3225Metric, symbol Device:C
- removed C23: .1uF, Capacitor_SMD:C_1210_3225Metric, symbol Device:C
- removed J15: HV_in_external, Connector_Coaxial:SMA_Molex_73251-2200_Horizontal, symbol Connector:Conn_Coaxial
- removed J17: SPI_right, Connector_PinHeader_2.54mm:PinHeader_1x06_P2.54mm_Vertical, symbol Connector_Generic:Conn_01x06
- removed J18: Measures_Digital, symbol Connector_Generic:Conn_01x04
- removed JP1: Jumper_3_Bridged12, symbol Jumper:Jumper_3_Bridged12
- removed JP2: VDD_JP, Connector_PinHeader_2.54mm:PinHeader_1x03_P2.54mm_Vertical, symbol Jumper:Jumper_3_Bridged12
- removed R9: 1k, Resistor_SMD:R_0603_1608Metric, symbol Device:R
- added C1, C6, C8: 1nF, Capacitor_SMD:C_0603_1608Metric, symbol Device:C
- added C10, C2, C9: .1uF, Capacitor_SMD:C_0603_1608Metric, symbol Device:C
- added C11, C13, C4: 10uF, Capacitor_SMD:C_0603_1608Metric, symbol Device:C
- added C14: 1nF, Capacitor_SMD:C_1210_3225Metric, symbol Device:C
- added C15: .1uF, Capacitor_SMD:C_1210_3225Metric, symbol Device:C
- added J1, J4: HBOut, Connector_Coaxial:SMA_Molex_73251-2200_Horizontal, symbol Connector:Conn_Coaxial
- added J7: HV_in_external, Connector_Coaxial:SMA_Molex_73251-2200_Horizontal, symbol Connector:Conn_Coaxial
- added J8: Conn_01x03, Connector_PinHeader_2.54mm:PinHeader_1x03_P2.54mm_Vertical, symbol Connector_Generic:Conn_01x03
- added R2, R3: 2k2, Resistor_SMD:R_0603_1608Metric, symbol Device:R
- added R4: 10k, Resistor_SMD:R_0603_1608Metric, symbol Device:R
- J12: footprint (none) -> Connector_PinHeader_2.54mm:PinHeader_1x04_P2.54mm_Vertical
- J13: footprint astropix:pcie_astropix -> Connector_PCBEdge:BUS_PCIexpress_x16
- J14: footprint (none) -> Connector_PinHeader_2.54mm:PinHeader_1x12_P2.54mm_Horizontal
- J2: footprint (none) -> Connector_PinHeader_2.54mm:PinHeader_1x05_P2.54mm_Vertical
- JP3: footprint (none) -> Connector_PinHeader_2.54mm:PinHeader_1x03_P2.54mm_Vertical
- JP4, JP5: footprint (none) -> Connector_PinHeader_2.54mm:PinHeader_1x02_P2.54mm_Vertical
- R1: value 10k -> 1k
- R6: value 0 -> 10k
- TP1, TP2: footprint (none) -> TestPoint:TestPoint_Loop_D1.80mm_Drill1.0mm_Beaded
- U2: footprint astropix:AstroPix5 -> astropix:AstroPix5_v2
Connections:
- net POW4_in is gone; now on net VDD: J13.B5 (POW4), J13.B6 (POW4)
- net clk20_Ext_N is gone; now on net Clk20_Ext_N: J13.B17 (FMC_LA24_N)
- net clk20_Ext_P is gone; now on net Clk20_Ext_P: J13.B16 (FMC_LA24_P)
- net GND: now also JP4.1 (A), JP5.1 (A), U2.GNDA_Ring (gnda!), U2.GND_Ring (gnd!), C1.2, C10.2, C11.2, C13.2, C14.1, C15.1, C2.2, C4.2, C6.2, C8.2, C9.2, J1.2 (Ext), J4.2 (Ext), J7.2 (Ext), J8.3 (Pin_3), R2.2, R3.2; no longer U2.B100 (gnda!), U2.B101 (gnda!), U2.B103 (gnda!), U2.B105 (gnda!), U2.B110 (gnd!), U2.B12 (gnda!), U2.B14 (gnda!), U2.B16 (gnda!), U2.B2 (gnd!), U2.B27 (gnd!), U2.B32 (gnd!), U2.B39 (gnd!), U2.B45 (gnd!), U2.B59 (gnd!), U2.B61 (gnda!), U2.B65 (gnda!), U2.B70 (gnda!), U2.B73 (gnda!), U2.B75 (gnda!), U2.B8 (gnd!), U2.B83 (gnda!), U2.B89 (gnda!), U2.B9 (gnd!), U2.B92 (gnda!), U2.B95 (gnd!)
- net HV_in_ext: now also R1.1, J7.1 (In)
- net ThPix: now also J14.6 (Pin_6), U2.B74 (ThPix)
- net VCasc2!: now also J14.8 (Pin_8), U2.B81 (VCasc2!)
- net VDD: now also U2.VDD_Ring (vdd!), C1.1, C2.1, C4.1, R4.2; no longer R1.1, U2.B1 (vdd!), U2.B10 (vdd!), U2.B109 (vdd!), U2.B11 (vdd!), U2.B26 (vdd!), U2.B44 (vdd!), U2.B58 (vdd!), U2.B94 (vdd!)
- net VDDA: now also U2.VDDA_Ring (vdda!), C10.1, C13.1, C8.1; no longer U2.B102 (vdda!), U2.B104 (vdda!), U2.B106 (vdda!), U2.B13 (vdda!), U2.B15 (vdda!), U2.B17 (vdda!), U2.B60 (vdda!), U2.B64 (vdda!), U2.B71 (vdda!), U2.B76 (vdda!), U2.B82 (vdda!), U2.B88 (vdda!), U2.B91 (vdda!), U2.B99 (vdda!)
- net VSSA: now also U2.VSSA_Ring (vssa!), C11.1, C6.1, C9.1; no longer U2.B107 (vssa!), U2.B108 (vssa!), U2.B18 (vssa!), U2.B19 (vssa!), U2.B62 (vssa!), U2.B63 (vssa!), U2.B80 (vssa!), U2.B87 (vssa!), U2.B90 (vssa!)
- net blpix: now also J14.2 (Pin_2), U2.B68 (blpix)
- net interrupt: now also J8.1 (Pin_1), R4.1; no longer R1.2
- net at U2.B24 (pll_clk): now also J4.1 (In)
- net suba: now reaches U2.B4 (sub!), U2.B5 (sub!)
- net suba: now also R1.2, C14.2, C15.2; no longer JP4.1 (A), JP5.1 (A)
- net at U2.B40 (HBOut): now also J5.1 (In), R3.1
- net at U2.B77 (ampout): now also J1.1 (In), R2.1
- net VDD18_in: no longer names the net of J13.B3 (VDD18)
- net VDD18_in: no longer J13.B4 (VDD18)
- no-connect marks 46 -> 53
Other:
- note added: "ni"
- moved on the sheet: J3, J5
